Commit message: work done

File: tacocat_description/urdf/camera.xacro (robot description, xacro)
@@ -1,5 +1,5 @@
 <?xml version="1.0"?>
 <robot name = "tacocat_camera" xmlns:xacro="http://www.ros.org/wiki/xacro">
-    <xacro:macro name="camera" params="">
+    <xacro:macro name="tacocam" params="">
         <link name="camera_link">
             <visual>
@@ -16,17 +16,18 @@
             <child link="camera_link"/>
         </joint>
-            <!-- camera -->
-    <gazebo reference="camera_link">
-        <sensor type="camera" name="camera1">
-            <update_rate>30.0</update_rate>
+    <!-- camera -->
+        <gazebo reference="camera_link">
+            <material>Gazebo/Black</material>
+            <sensor type="camera" name="camera1">
+            <update_rate>60.0</update_rate>
             <camera name="head">
-                <horizontal_fov>1.3962634</horizontal_fov>
+                <horizontal_fov>1.5708</horizontal_fov>
                 <image>
-                    <width>800</width>
-                    <height>800</height>
+                    <width>2560</width>
+                    <height>720</height>
                     <format>R8G8B8</format>
                 </image>
                 <clip>
-                    <near>0.02</near>
+                    <near>0.035</near>
                     <far>300</far>
                 </clip>
@@ -43,6 +44,6 @@
                 <alwaysOn>true</alwaysOn>
                 <updateRate>0.0</updateRate>
-                <cameraName>tacocat/camera1</cameraName>
-                <imageTopicName>image_raw</imageTopicName>
+                <cameraName>tacocat/tacocam</cameraName>
+                <imageTopicName>image</imageTopicName>
                 <cameraInfoTopicName>camera_info</cameraInfoTopicName>
                 <frameName>camera_link</frameName>
@@ -54,6 +55,6 @@
                 <distortionT2>0.0</distortionT2>
             </plugin>
-        </sensor>
-    </gazebo>
+            </sensor>
+        </gazebo>
     </xacro:macro>
 </robot>

File: tacocat_description/urdf/tacocat.xacro (robot description, xacro)
@@ -5,6 +5,8 @@
     <xacro:include filename="$(find tacocat_description)/urdf/wheel.xacro"/>
     <xacro:include filename="$(find tacocat_description)/urdf/camera.xacro"/>
+    <xacro:include filename="$(find tacocat_description)/urdf/laser.xacro"/>
     <xacro:chassis/>
-    <xacro:camera/>
+    <xacro:tacocam/>
+    <xacro:laser/>
     <xacro:wheel
         name="left"
